File: hardware/elka.brd (EAGLE design)
At the start: 50 x 50 mm, 57 parts

Commit message: Окончательный (надеюсь) вариант трассировки
Parts:
- removed R22: 910, common-rcl:SMD0603
- removed TP18: TPSQTP20R, testpad:TP20R
- added C10, C9: 0.1u, common-rcl:SMD0603
- added DA2: ADP3338AKCZ-3.3RL7, analog-devices:SOT223-W
- added R24, R25, R26, R27: 910, common-rcl:SMD0603
- added S1: DPDT-6, other:DPDT
- added TP24: TPSQTP20R, testpad:TP20R
- C1: value 10u -> 0.01u; device common-rcl:SMC_B -> common-rcl:SMD0603
- C3, C8: value 0.1u -> 10u; device common-rcl:SMD0603 -> common-rcl:SMC_B
- C6: value 10u -> 0.1u; device common-rcl:SMC_B -> common-rcl:SMD0603
- DA1: value ADP3338AKCZ-3.3RL7 -> LM358ADR; device analog-devices:SOT223-W -> texas-instruments:SOIC8
- R1, R12: value 910 -> 1k
- R10: value 910 -> 62k
- R11, R2, R20, R21: value 910 -> 10k
- R16, R17, R8: value 10k -> 910
- moved C2 37.5 mm to (44.0, 41.8), turned to 180 degrees
- moved C6 35.2 mm to (22.9, 39.4), turned to 225 degrees
- moved C1 33.0 mm to (35.4, 42.9), turned to 45 degrees
- moved DA1 29.5 mm to (40.5, 38.5), turned to 270 degrees
- moved R21 27.4 mm to (42.1, 42.4), turned to 270 degrees
- moved C5 24.7 mm to (22.1, 29.9), turned to 45 degrees
- moved R8 23.1 mm to (28.8, 38.3), turned to 45 degrees
- moved C4 21.5 mm to (39.9, 26.2), turned to 180 degrees
- moved C3 18.8 mm to (39.8, 23.4), turned to 180 degrees
- moved R17 18.2 mm to (17.6, 38.9), turned to 135 degrees
- moved R11 15.8 mm to (6.45, 32.4), turned to 270 degrees
- moved R12 14.8 mm to (32.0, 46.4), turned to 315 degrees
- moved R10 14.6 mm to (35.9, 39.8), turned to 270 degrees
- moved C8 13.9 mm to (38.0, 30.0), turned to 270 degrees
- moved R2 13.4 mm to (38.7, 42.2), turned to 0 degrees
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Connections:
- removed net LED14: DD1.15, R18.1
- new net ADC: DD1.15, R12.1
- new net N$2: C1.1, DA1.3, R1.1
- new net N$26: R1.2, TP24.TP
- new net N$7: DA1.2, R10.2, R2.2
- new net N$9: DA1.1, R10.1, R12.2
- net !NRST: now also R20.1; no longer R16.1
- net +3.3V: now also C2.2, C5.2, C6.2, C7.1, C8.+, C9.2, DA1.8, DA2.2, DA2.4, R20.2, R21.2; no longer C3.2, C4.2, C5.1, C6.+, C7.2, DA1.2, DA1.4, R16.2, R17.2
- net +4.5V: now also S1.3, S1.4, S1.5, S1.6; no longer C1.+, C2.1, DA1.3
- net GND: now also C1.2, C10.2, C2.1, C3.-, C4.2, C5.1, C6.1, C7.2, C8.-, C9.1, DA1.4, DA1.5, DA1.6, DA2.1, R11.2, R2.1; no longer C1.-, C2.2, C3.1, C4.1, C5.2, C6.-, C7.1, C8.2, DA1.1, R8.2
- net LED0: now also R3.1; no longer R1.1
- net LED1: now also R4.1; no longer R2.1
- net LED10: now also R16.1; no longer R12.1
- net LED11: now also R17.1; no longer R13.1
- net LED12: now also R18.1; no longer R14.1
- net LED13: now also R19.1; no longer R15.1
- net LED15: now also R23.1; no longer R19.1
- net LED16: now also R24.1; no longer R20.1
- net LED17: now also R25.1; no longer R21.1
- net LED18: now also R26.1; no longer R22.1
- net LED19: now also R27.1; no longer R23.1
- net LED2: now also R5.1; no longer R3.1
- net LED3: now also R6.1; no longer R4.1
- net LED4: now also R7.1; no longer R5.1
- net LED5: now also R8.1; no longer R6.1
- net LED6: now also R9.1; no longer R7.1
- net LED7: now also R13.1; no longer R9.1
- net LED8: now also R14.1; no longer R10.1
- net LED9: now also R15.1; no longer R11.1
- net N$1: now also R14.2; no longer R10.2
- net N$10: now also R3.2; no longer R1.2
- net N$11: now also R4.2; no longer R2.2
- net N$12: now also R5.2; no longer R3.2
- net N$13: now also R6.2; no longer R4.2
- net N$14: now also R7.2; no longer R5.2
- net N$15: now also R8.2; no longer R6.2
- net N$16: now also R13.2; no longer R9.2
- net N$17: now also R9.2; no longer R7.2
- net N$18: now also C3.+, C4.1, DA2.3, S1.1, S1.2; no longer R18.2, TP18.TP
- net N$19: now also R23.2; no longer R19.2
- net N$20: now also R24.2; no longer R20.2
- net N$21: now also R25.2; no longer R21.2
- net N$22: now also R26.2; no longer R22.2
- net N$23: now also R27.2; no longer R23.2
- net N$24: now also C10.1, R21.1; no longer C8.1, R17.1
- net N$3: now also R15.2; no longer R11.2
- net N$4: now also R16.2; no longer R12.2
- net N$5: now also R17.2; no longer R13.2
- net N$6: now also R18.2; no longer R14.2
- net N$8: now also R19.2; no longer R15.2
- net SWCLK: now also R11.1; no longer R8.1
Routing:
- net ADC: track 0.00 -> 17.0 mm
- net N$18: track 4.05 -> 18.9 mm
- net +4.5V: track 5.49 -> 14.7 mm
- net N$9: track 0.00 -> 8.67 mm
- net N$2: track 0.00 -> 7.99 mm
- net N$7: track 0.00 -> 6.62 mm
- net +3.3V: track 69.9 -> 65.8 mm
- net LED14: track 3.96 -> 0.00 mm
- net LED18: track 3.77 -> 6.40 mm
- net N$22: track 3.21 -> 5.60 mm
- net N$23: track 2.28 -> 4.61 mm
- net N$24: track 33.0 -> 30.9 mm
- net N$26: track 0.00 -> 1.88 mm
- net LED15: track 3.15 -> 4.93 mm
- net GND: track 15.1 -> 16.7 mm
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- added copper zone on layer 1, net +4.5V
- added copper zone on layer 1, net N$18
Other:
- board text added: "Happy New Year!"
- board text removed: "Happy New Year! 2017"
