File: hardware/elka.sch (EAGLE design)
At the start: 57 parts

Commit message: Окончательный (надеюсь) вариант трассировки
Parts:
- removed TP18: TPSQTP20R, testpad:TPSQTP20R
- added C10, C9: 0.1u, common-rcl:C0603
- added DA2: ADP3338AKCZ-3.3RL7, analog-devices:ADP3338AKCZ-3.3RL7
- added R24, R25, R27: 910, common-rcl:R0603
- added S1: DPDT-6, other:DPDT-6
- added TP24: TPSQTP20R, testpad:TPSQTP20R
- C1: value 10u -> 0.01u; device common-rcl:CPOLSMC_B -> common-rcl:C0603
- C3, C8: value 0.1u -> 10u; device common-rcl:C0603 -> common-rcl:CPOLSMC_B
- C6: value 10u -> 0.1u; device common-rcl:CPOLSMC_B -> common-rcl:C0603
- DA1: value ADP3338AKCZ-3.3RL7 -> LM358ADR; device analog-devices:ADP3338AKCZ-3.3RL7 -> texas-instruments:LM358ADR
- R1, R12: value 910 -> 1k
- R10: value 910 -> 62k
- R11, R2, R20, R21: value 910 -> 10k
- R16, R17, R8: value 10k -> 910
- renumbered R22 to R26
Connections:
- removed net LED14: DD1.PB1, R18.1
- new net ADC: DD1.PB1, R12.1
- new net N$2: C1.1, DA1.1.IN+, R1.1
- new net N$26: R1.2, TP24.TP
- new net N$7: DA1.1.IN-, R10.2, R2.2
- new net N$9: DA1.1.OUT, R10.1, R12.2
- net !NRST: now also R20.1; no longer R16.1
- net +3.3V: now also C2.2, C5.2, C6.2, C7.1, C8.+, C9.2, DA1G$3.VCC+, DA2.OUT@1, DA2.OUT@2, R20.2, R21.2; no longer C3.2, C4.2, C5.1, C6.+, C7.2, DA1.OUT@1, DA1.OUT@2, R16.2, R17.2
- net +4.5V: now also S1.3, S1.4, S1.5, S1.6; no longer C1.+, C2.1, DA1.IN
- net GND: now also C1.2, C10.2, C2.1, C3.-, C4.2, C5.1, C6.1, C7.2, C8.-, C9.1, DA1.2.IN+, DA1.2.IN-, DA1G$3.VCC-, DA2.GND, R11.2, R2.1; no longer C1.-, C2.2, C3.1, C4.1, C5.2, C6.-, C7.1, C8.2, DA1.GND, R8.2
- net LED0: now also R3.1; no longer R1.1
- net LED1: now also R4.1; no longer R2.1
- net LED10: now also R16.1; no longer R12.1
- net LED11: now also R17.1; no longer R13.1
- net LED12: now also R18.1; no longer R14.1
- net LED13: now also R19.1; no longer R15.1
- net LED15: now also R23.1; no longer R19.1
- net LED16: now also R24.1; no longer R20.1
- net LED17: now also R25.1; no longer R21.1
- net LED19: now also R27.1; no longer R23.1
- net LED2: now also R5.1; no longer R3.1
- net LED3: now also R6.1; no longer R4.1
- net LED4: now also R7.1; no longer R5.1
- net LED5: now also R8.1; no longer R6.1
- net LED6: now also R9.1; no longer R7.1
- net LED7: now also R13.1; no longer R9.1
- net LED8: now also R14.1; no longer R10.1
- net LED9: now also R15.1; no longer R11.1
- net N$1: now also R14.2; no longer R10.2
- net N$10: now also R3.2; no longer R1.2
- net N$11: now also R4.2; no longer R2.2
- net N$12: now also R5.2; no longer R3.2
- net N$13: now also R6.2; no longer R4.2
- net N$14: now also R7.2; no longer R5.2
- net N$15: now also R8.2; no longer R6.2
- net N$16: now also R13.2; no longer R9.2
- net N$17: now also R9.2; no longer R7.2
- net N$18: now also C3.+, C4.1, DA2.IN, S1.1, S1.2; no longer R18.2, TP18.TP
- net N$19: now also R23.2; no longer R19.2
- net N$20: now also R24.2; no longer R20.2
- net N$21: now also R25.2; no longer R21.2
- net N$23: now also R27.2; no longer R23.2
- net N$24: now also C10.1, R21.1; no longer C8.1, R17.1
- net N$3: now also R15.2; no longer R11.2
- net N$4: now also R16.2; no longer R12.2
- net N$5: now also R17.2; no longer R13.2
- net N$6: now also R18.2; no longer R14.2
- net N$8: now also R19.2; no longer R15.2
- net SWCLK: now also R11.1; no longer R8.1
Other:
- note added: "PB2-PB6"
- note added: "PB7"
- note removed: "PB1-PB5"
- note removed: "PB6"
- moved on the sheet: C2, C4, C5, C7, R1, R10, R11, R12, R13, R14, R15, R16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
